File: Main_Board/kicad_project/power.sch (KiCad schematic (older format))
At the start: 32 parts, among them J5 PWR_ENTRY, J6 12V_HDR, J7 3V3_HDR, J8 5V_HDR, U5 TPS562200, U6 TPS562200

Commit message: progress on MCU pinout
Parts:
- renumbered C45 to C?, C47 to C?, C49 to C?, C51 to C?, C53 to C?, C43 to C?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

Commit message: progress?
Parts:
- gave numbers to parts that had none: 32
