File: Main_Board/kicad_project/limit_sw.sch (KiCad schematic (older format))
At the start: 70 parts

Commit message: progress?
Parts:
- gave numbers to parts that had none: 70

Commit message: progress on MCU pinout
Parts:
- renumbered C63 to C?, C64 to C?, C68 to C?, C67 to C?, C71 to C?, C72 to C?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
