File: Main_Board/kicad_project/expansion.sch (KiCad schematic (older format))
At the start: 0 parts

Commit message: schematic rev1 finished
Parts:
- added D20, D21, D22, D23, D24, D25, D26, D27, D28, D29, D30, D31, D32, D33, D34: PESD3V3S2UT, Package_TO_SOT_SMD:SOT-23, symbol Device:D_Zener_x2_ACom_KKA
- added J24: EXPANSION_HEADER, Connector_IDC:IDC-Header_2x20_P2.54mm_Vertical, symbol Connector_Generic:Conn_02x20_Odd_Even
- added RN1, RN2, RN3, RN4, RN5, RN6, RN7, RN8: 150R, Resistor_SMD:R_Array_Convex_4x1206, symbol Device:R_Pack04
Connections:
- net EXP_IO1: now also D20.1 (K), RN1.1 (R1.1)
- net EXP_IO10: now also D21.2 (K), RN3.2 (R2.1)
- net EXP_IO11: now also D25.1 (K), RN3.3 (R3.1)
- net EXP_IO12: now also D25.2 (K), RN3.4 (R4.1)
- net EXP_IO13: now also D29.1 (K), RN4.1 (R1.1)
- net EXP_IO14: now also D29.2 (K), RN4.2 (R2.1)
- net EXP_IO15: now also D33.1 (K), RN4.3 (R3.1)
- net EXP_IO16: now also D22.1 (K), RN5.1 (R1.1)
- net EXP_IO17: now also D22.2 (K), RN5.2 (R2.1)
- net EXP_IO18: now also D26.1 (K), RN5.3 (R3.1)
- net EXP_IO19: now also D26.2 (K), RN5.4 (R4.1)
- net EXP_IO2: now also D20.2 (K), RN1.2 (R2.1)
- net EXP_IO20: now also D30.1 (K), RN6.1 (R1.1)
- net EXP_IO21: now also D30.2 (K), RN6.2 (R2.1)
- net EXP_IO22: now also D34.1 (K), RN6.3 (R3.1)
- net EXP_IO23: now also D34.2 (K), RN6.4 (R4.1)
- net EXP_IO24: now also D23.1 (K), RN7.1 (R1.1)
- net EXP_IO25: now also D23.2 (K), RN7.2 (R2.1)
- net EXP_IO26: now also D27.1 (K), RN7.3 (R3.1)
- net EXP_IO27: now also D27.2 (K), RN7.4 (R4.1)
- net EXP_IO28: now also D31.1 (K), RN8.1 (R1.1)
- net EXP_IO29: now also D31.2 (K), RN8.2 (R2.1)
- net EXP_IO3: now also D24.1 (K), RN1.3 (R3.1)
- net EXP_IO30: now also D33.2 (K), RN8.3 (R3.1)
- net EXP_IO4: now also D24.2 (K), RN1.4 (R4.1)
- net EXP_IO5: now also D28.1 (K), RN2.1 (R1.1)
- net EXP_IO6: now also D28.2 (K), RN2.2 (R2.1)
- net EXP_IO7: now also D32.1 (K), RN2.3 (R3.1)
- net EXP_IO8: now also D32.2 (K), RN2.4 (R4.1)
- net EXP_IO9: now also D21.1 (K), RN3.1 (R1.1)
- new net: J24.10 (Pin_10), RN5.6 (R3.2)
- new net: J24.11 (Pin_11), RN1.5 (R4.2)
- new net: J24.12 (Pin_12), RN5.5 (R4.2)
- new net: J24.13 (Pin_13), RN2.8 (R1.2)
- new net: J24.14 (Pin_14), RN6.8 (R1.2)
- new net: J24.17 (Pin_17), RN2.7 (R2.2)
- new net: J24.18 (Pin_18), RN6.7 (R2.2)
- new net: J24.19 (Pin_19), RN2.6 (R3.2)
- new net: J24.20 (Pin_20), RN6.6 (R3.2)
- new net: J24.21 (Pin_21), RN2.5 (R4.2)
- new net: J24.22 (Pin_22), RN6.5 (R4.2)
- new net: J24.23 (Pin_23), RN3.8 (R1.2)
- new net: J24.24 (Pin_24), RN7.8 (R1.2)
- new net: J24.25 (Pin_25), RN3.7 (R2.2)
- new net: J24.26 (Pin_26), RN7.7 (R2.2)
- new net: J24.29 (Pin_29), RN3.6 (R3.2)
- new net: J24.30 (Pin_30), RN7.6 (R3.2)
- new net: J24.31 (Pin_31), RN3.5 (R4.2)
- new net: J24.32 (Pin_32), RN7.5 (R4.2)
- new net: J24.33 (Pin_33), RN4.8 (R1.2)
- new net: J24.34 (Pin_34), RN8.8 (R1.2)
- new net: J24.35 (Pin_35), RN4.7 (R2.2)
- new net: J24.36 (Pin_36), RN8.7 (R2.2)
- new net: J24.37 (Pin_37), RN4.6 (R3.2)
- new net: J24.38 (Pin_38), RN8.6 (R3.2)
- new net: J24.5 (Pin_5), RN1.8 (R1.2)
- new net: J24.6 (Pin_6), RN5.8 (R1.2)
- new net: J24.7 (Pin_7), RN1.7 (R2.2)
- new net: J24.8 (Pin_8), RN5.7 (R2.2)
- new net: J24.9 (Pin_9), RN1.6 (R3.2)
- new net 12V: J24.1 (Pin_1), J24.2 (Pin_2)
- new net 3V3: J24.3 (Pin_3), J24.4 (Pin_4)
- new net GND: D20.3 (A), D21.3 (A), D22.3 (A), D23.3 (A), D24.3 (A), D25.3 (A), D26.3 (A), D27.3 (A), D28.3 (A), D29.3 (A), D30.3 (A), D31.3 (A), D32.3 (A), D33.3 (A), D34.3 (A), J24.15 (Pin_15), J24.16 (Pin_16), J24.27 (Pin_27), J24.28 (Pin_28), J24.39 (Pin_39), J24.40 (Pin_40)
Other:
- note added: "Each signal pin protected with TVS diode and 150 ohm series resistor.\nConnector is IDC 40 pin, designed to have both cable or a board plugged into.\nPCB should include standoffs for larger expansion boards."
- note added: "Expansion Header"

Commit message: expansion connector - rev 1.1 schematic, finished layout
Parts:
- J24: symbol Connector_Generic:Conn_02x20_Odd_Even -> Connector_Generic:Conn_02x20_Top_Bottom
Connections:
- net EXP_IO1: now also RN1.4 (R4.1); no longer RN1.1 (R1.1)
- net EXP_IO10: now also RN3.3 (R3.1); no longer RN3.2 (R2.1)
- net EXP_IO11: now also RN3.2 (R2.1); no longer RN3.3 (R3.1)
- net EXP_IO12: now also RN3.1 (R1.1); no longer RN3.4 (R4.1)
- net EXP_IO13: now also RN4.4 (R4.1); no longer RN4.1 (R1.1)
- net EXP_IO14: now also RN4.3 (R3.1); no longer RN4.2 (R2.1)
- net EXP_IO15: now also RN5.4 (R4.1); no longer RN4.3 (R3.1)
- net EXP_IO16: now also D33.2 (K), RN5.3 (R3.1); no longer D22.1 (K), RN5.1 (R1.1)
- net EXP_IO17: now also D22.1 (K); no longer D22.2 (K)
- net EXP_IO18: now also D22.2 (K), RN5.1 (R1.1); no longer D26.1 (K), RN5.3 (R3.1)
- net EXP_IO19: now also D26.1 (K), RN6.4 (R4.1); no longer D26.2 (K), RN5.4 (R4.1)
- net EXP_IO2: now also RN1.3 (R3.1); no longer RN1.2 (R2.1)
- net EXP_IO20: now also D26.2 (K), RN6.3 (R3.1); no longer D30.1 (K), RN6.1 (R1.1)
- net EXP_IO21: now also D30.1 (K); no longer D30.2 (K)
- net EXP_IO22: now also D30.2 (K), RN6.1 (R1.1); no longer D34.1 (K), RN6.3 (R3.1)
- net EXP_IO23: now also D34.1 (K), RN7.4 (R4.1); no longer D34.2 (K), RN6.4 (R4.1)
- net EXP_IO24: now also D34.2 (K), RN7.3 (R3.1); no longer D23.1 (K), RN7.1 (R1.1)
- net EXP_IO25: now also D23.1 (K); no longer D23.2 (K)
- net EXP_IO26: now also D23.2 (K), RN7.1 (R1.1); no longer D27.1 (K), RN7.3 (R3.1)
- net EXP_IO27: now also D27.1 (K), RN8.4 (R4.1); no longer D27.2 (K), RN7.4 (R4.1)
- net EXP_IO28: now also D27.2 (K), RN8.3 (R3.1); no longer D31.1 (K), RN8.1 (R1.1)
- net EXP_IO29: now also D31.1 (K); no longer D31.2 (K)
- net EXP_IO3: now also RN1.2 (R2.1); no longer RN1.3 (R3.1)
- net EXP_IO30: now also D31.2 (K), RN8.1 (R1.1); no longer D33.2 (K), RN8.3 (R3.1)
- net EXP_IO4: now also RN1.1 (R1.1); no longer RN1.4 (R4.1)
- net EXP_IO5: now also RN2.4 (R4.1); no longer RN2.1 (R1.1)
- net EXP_IO6: now also RN2.3 (R3.1); no longer RN2.2 (R2.1)
- net EXP_IO7: now also RN2.2 (R2.1); no longer RN2.3 (R3.1)
- net EXP_IO8: now also RN2.1 (R1.1); no longer RN2.4 (R4.1)
- net EXP_IO9: now also RN3.4 (R4.1); no longer RN3.1 (R1.1)
- net at J24.10 (Pin_10): now also RN2.6 (R3.2); no longer RN5.6 (R3.2)
- net at J24.11 (Pin_11): now also RN2.7 (R2.2); no longer RN1.5 (R4.2)
- net at J24.12 (Pin_12): now also RN2.8 (R1.2); no longer RN5.5 (R4.2)
- net at J24.13 (Pin_13): now also RN3.5 (R4.2); no longer RN2.8 (R1.2)
- net at J24.14 (Pin_14): now also RN3.6 (R3.2); no longer RN6.8 (R1.2)
- net at J24.17 (Pin_17): now also RN3.7 (R2.2); no longer RN2.7 (R2.2)
- net at J24.18 (Pin_18): now also RN3.8 (R1.2); no longer RN6.7 (R2.2)
- net at J24.19 (Pin_19): now also RN4.5 (R4.2); no longer RN2.6 (R3.2)
- net at J24.20 (Pin_20): now also RN4.6 (R3.2); no longer RN6.6 (R3.2)
- net at J24.21 (Pin_21): now also RN5.5 (R4.2); no longer RN2.5 (R4.2)
- net at J24.22 (Pin_22): now also RN5.6 (R3.2); no longer RN6.5 (R4.2)
- net at J24.23 (Pin_23): now also RN5.7 (R2.2); no longer RN3.8 (R1.2)
- net at J24.24 (Pin_24): now also RN5.8 (R1.2); no longer RN7.8 (R1.2)
- net at J24.25 (Pin_25): now also RN6.5 (R4.2); no longer RN3.7 (R2.2)
- net at J24.26 (Pin_26): now also RN6.6 (R3.2); no longer RN7.7 (R2.2)
- net at J24.29 (Pin_29): now also RN6.7 (R2.2); no longer RN3.6 (R3.2)
- net at J24.30 (Pin_30): now also RN6.8 (R1.2); no longer RN7.6 (R3.2)
- net at J24.31 (Pin_31): now also RN7.5 (R4.2); no longer RN3.5 (R4.2)
- net at J24.32 (Pin_32): now also RN7.6 (R3.2); no longer RN7.5 (R4.2)
- net at J24.33 (Pin_33): now also RN7.7 (R2.2); no longer RN4.8 (R1.2)
- net at J24.34 (Pin_34): now also RN7.8 (R1.2); no longer RN8.8 (R1.2)
- net at J24.35 (Pin_35): now also RN8.5 (R4.2); no longer RN4.7 (R2.2)
- net at J24.36 (Pin_36): now also RN8.6 (R3.2); no longer RN8.7 (R2.2)
- net at J24.37 (Pin_37): now also RN8.7 (R2.2); no longer RN4.6 (R3.2)
- net at J24.38 (Pin_38): now also RN8.8 (R1.2); no longer RN8.6 (R3.2)
- net at J24.5 (Pin_5): now also RN1.5 (R4.2); no longer RN1.8 (R1.2)
- net at J24.6 (Pin_6): now also RN1.6 (R3.2); no longer RN5.8 (R1.2)
- net at J24.8 (Pin_8): now also RN1.8 (R1.2); no longer RN5.7 (R2.2)
- net at J24.9 (Pin_9): now also RN2.5 (R4.2); no longer RN1.6 (R3.2)
Other:
- moved on the sheet: RN1, RN2, RN3, RN4, RN5, RN6, RN7, RN8
