File: Main_Board/kicad_project/external_io.sch (KiCad schematic (older format))
At the start: 19 parts

Commit message: progress?
Parts:
- gave numbers to parts that had none: 19
Changed lines of the file:
@@
 $EndDescr
 $Comp
-L Interface:PCA9600DP U?
+L Interface:PCA9600DP U8
 U 1 1 5F70BE3C
 P 5875 4200
-F 0 "U?" H 5725 3850 50  0000 C CNN
+F 0 "U8" H 5725 3850 50  0000 C CNN
 F 1 "PCA9600DP" H 6200 3850 50  0000 C CNN
 F 2 "Package_SO:TSSOP-8_3x3mm_P0.65mm" H 6675 3850 50  0001 C CNN
@@
 $EndComp
 $Comp
-L Connector:USB_B_Micro J?
+L Connector:USB_B_Micro J20
 U 1 1 5F70DEC7
 P 4775 1675
-F 0 "J?" H 4950 1300 50  0000 C CNN
+F 0 "J20" H 4950 1300 50  0000 C CNN
 F 1 "USB_B_Micro" H 4832 2051 50  0000 C CNN
 F 2 "Connector_USB:USB_Micro-B_Molex_47346-0001" H 4925 1625 50  0001 C CNN
@@
 $EndComp
 $Comp
-L LoaDy:USBLC6-2SC6 U?
+L LoaDy:USBLC6-2SC6 U9
 U 1 1 5F71A98E
 P 6450 1725
-F 0 "U?" H 6450 2192 50  0000 C CNN
+F 0 "U9" H 6450 2192 50  0000 C CNN
 F 1 "USBLC6-2SC6" H 6450 2101 50  0000 C CNN
 F 2 "Package_TO_SOT_SMD:SOT-23-6" H 7275 2125 50  0001 C CNN
@@
 $EndComp
 $Comp
-L power:GND #PWR?
+L power:GND #PWR081
 U 1 1 5F71E77C
 P 4775 2400
-F 0 "#PWR?" H 4775 2150 50  0001 C CNN
+F 0 "#PWR081" H 4775 2150 50  0001 C CNN
 F 1 "GND" H 4780 2227 50  0000 C CNN
 F 2 "" H 4775 2400 50  0001 C CNN
@@
 	5425 1725 5425 1475
 $Comp
-L Device:R_Small R?
+L Device:R_Small R55
 U 1 1 5F7222AA
 P 4675 2225
-F 0 "R?" H 4617 2179 50  0000 R CNN
+F 0 "R55" H 4617 2179 50  0000 R CNN
 F 1 "33K" H 4617 2270 50  0000 R CNN
 F 2 "Resistor_SMD:R_0603_1608Metric" H 4675 2225 50  0001 C CNN
@@
 	4675 2125 4675 2075
 $Comp
-L power:GND #PWR?
+L power:GND #PWR088
 U 1 1 5F72339E
 P 7000 1725
-F 0 "#PWR?" H 7000 1475 50  0001 C CNN
+F 0 "#PWR088" H 7000 1475 50  0001 C CNN
 F 1 "GND" V 7005 1597 50  0000 R CNN
 F 2 "" H 7000 1725 50  0001 C CNN
@@
 USB_DP
 $Comp
-L Device:R_Small R?
+L Device:R_Small R60
 U 1 1 5F728398
 P 7650 4100
-F 0 "R?" V 7700 3975 50  0000 C CNN
+F 0 "R60" V 7700 3975 50  0000 C CNN
 F 1 "0R" V 7600 4225 50  0000 C CNN
 F 2 "Resistor_SMD:R_0603_1608Metric" H 7650 4100 50  0001 C CNN
@@
 $EndComp
 $Comp
-L Device:R_Small R?
+L Device:R_Small R61
 U 1 1 5F728F58
 P 7650 4300
-F 0 "R?" V 7700 4175 50  0000 C CNN
+F 0 "R61" V 7700 4175 50  0000 C CNN
 F 1 "0R" V 7600 4425 50  0000 C CNN
 F 2 "Resistor_SMD:R_0603_1608Metric" H 7650 4300 50  0001 C CNN
@@
 	7550 4300 7475 4300
 $Comp
-L Device:Jumper_NO_Small JP?
+L Device:Jumper_NO_Small JP1
 U 1 1 5F730E54
 P 7650 3950
-F 0 "JP?" H 7650 4100 50  0000 C CNN
+F 0 "JP1" H 7650 4100 50  0000 C CNN
 F 1 "SDA_JMP" H 7650 4025 50  0000 C CNN
 F 2 "Connector_PinHeader_2.54mm:PinHeader_1x02_P2.54mm_Vertical" H 7650 3950 50  0001 C CNN
@@
 $EndComp
 $Comp
-L Device:Jumper_NO_Small JP?
+L Device:Jumper_NO_Small JP2
 U 1 1 5F7312C9
 P 7650 4450
-F 0 "JP?" H 7650 4600 50  0000 C CNN
+F 0 "JP2" H 7650 4600 50  0000 C CNN
 F 1 "SCL_JMP" H 7650 4525 50  0000 C CNN
 F 2 "Connector_PinHeader_2.54mm:PinHeader_1x02_P2.54mm_Vertical" H 7650 4450 50  0001 C CNN
@@
 3V3
 $Comp
-L power:GND #PWR?
+L power:GND #PWR086
 U 1 1 5F72CC53
 P 6450 3875
-F 0 "#PWR?" H 6450 3625 50  0001 C CNN
+F 0 "#PWR086" H 6450 3625 50  0001 C CNN
 F 1 "GND" H 6455 3702 50  0000 C CNN
 F 2 "" H 6450 3875 50  0001 C CNN
@@
 $EndComp
 $Comp
-L Connector_Generic:Conn_01x04 J?
+L Connector_Generic:Conn_01x04 J22
 U 1 1 5F729670
 P 6225 3650
-F 0 "J?" H 6350 3750 50  0000 C CNN
+F 0 "J22" H 6350 3750 50  0000 C CNN
 F 1 "I2C_EXTERNAL" H 6143 3876 50  0000 C CNN
 F 2 "Connector_PinHeader_2.54mm:PinHeader_1x04_P2.54mm_Vertical" H 6225 3650 50  0001 C CNN
@@
 	6675 4300 7000 4300
 $Comp
-L Device:R_Small R?
+L Device:R_Small R58
 U 1 1 5F74371A
 P 7000 3925
-F 0 "R?" H 6950 3875 50  0000 R CNN
+F 0 "R58" H 6950 3875 50  0000 R CNN
 F 1 "4K7" H 6950 3975 50  0000 R CNN
 F 2 "Resistor_SMD:R_0603_1608Metric" H 7000 3925 50  0001 C CNN
@@
 $EndComp
 $Comp
-L Device:R_Small R?
+L Device:R_Small R59
 U 1 1 5F743EA7
 P 7100 3925
-F 0 "R?" H 7050 3875 50  0000 R CNN
+F 0 "R59" H 7050 3875 50  0000 R CNN
 F 1 "4K7" H 7050 3975 50  0000 R CNN
 F 2 "Resistor_SMD:R_0603_1608Metric" H 7100 3925 50  0001 C CNN
@@
 Connection ~ 7100 3725
 $Comp
-L power:GND #PWR?
+L power:GND #PWR084
 U 1 1 5F747299
 P 5875 4600
-F 0 "#PWR?" H 5875 4350 50  0001 C CNN
+F 0 "#PWR084" H 5875 4350 50  0001 C CNN
 F 1 "GND" H 5880 4427 50  0000 C CNN
 F 2 "" H 5875 4600 50  0001 C CNN
@@
 $EndComp
 $Comp
-L Connector_Generic:Conn_01x04 J?
+L Connector_Generic:Conn_01x04 J19
 U 1 1 5F7475E6
 P 3925 4150
-F 0 "J?" H 3900 3825 50  0000 C CNN
+F 0 "J19" H 3900 3825 50  0000 C CNN
 F 1 "I2C_BUFFERED" H 4000 4375 50  0000 C CNN
 F 2 "Connector_PinHeader_2.54mm:PinHeader_1x04_P2.54mm_Horizontal" H 3925 4150 50  0001 C CNN
@@
 Connection ~ 5525 4100
 $Comp
-L Device:C_Small C?
+L Device:C_Small C73
 U 1 1 5F74C7A6
 P 5625 3575
-F 0 "C?" H 5650 3650 50  0000 L CNN
+F 0 "C73" H 5650 3650 50  0000 L CNN
 F 1 "100n" H 5650 3500 50  0000 L CNN
 F 2 "Capacitor_SMD:C_0603_1608Metric" H 5625 3575 50  0001 C CNN
@@
 $EndComp
 $Comp
-L power:GND #PWR?
+L power:GND #PWR083
 U 1 1 5F74C9C7
 P 5625 3675
-F 0 "#PWR?" H 5625 3425 50  0001 C CNN
+F 0 "#PWR083" H 5625 3425 50  0001 C CNN
 F 1 "GND" H 5630 3502 50  0000 C CNN
 F 2 "" H 5625 3675 50  0001 C CNN
@@
 $EndComp
 $Comp
-L Device:R_Small R?
+L Device:R_Small R57
 U 1 1 5F74F68F
 P 5225 3800
-F 0 "R?" H 5175 3750 50  0000 R CNN
+F 0 "R57" H 5175 3750 50  0000 R CNN
 F 1 "2K2" H 5175 3850 50  0000 R CNN
 F 2 "Resistor_SMD:R_0603_1608Metric" H 5225 3800 50  0001 C CNN
@@
 $EndComp
 $Comp
-L Device:R_Small R?
+L Device:R_Small R56
 U 1 1 5F74FC84
 P 5125 3800
-F 0 "R?" H 5075 3750 50  0000 R CNN
+F 0 "R56" H 5075 3750 50  0000 R CNN
 F 1 "2K2" H 5075 3850 50  0000 R CNN
 F 2 "Resistor_SMD:R_0603_1608Metric" H 5125 3800 50  0001 C CNN
@@
 	4150 4375 4150 4350
 $Comp
-L power:GND #PWR?
+L power:GND #PWR079
 U 1 1 5F76116E
 P 4150 4375
-F 0 "#PWR?" H 4150 4125 50  0001 C CNN
+F 0 "#PWR079" H 4150 4125 50  0001 C CNN
 F 1 "GND" H 4155 4202 50  0000 C CNN
 F 2 "" H 4150 4375 50  0001 C CNN
@@
 P 4700 4475
 AR Path="/5F51A37F/5F783DBC" Ref="D?"  Part="1"
-AR Path="/5F709561/5F783DBC" Ref="D?"  Part="1"
-F 0 "D?" H 4600 4375 50  0000 C CNN
+AR Path="/5F709561/5F783DBC" Ref="D11"  Part="1"
+F 0 "D11" H 4600 4375 50  0000 C CNN
 F 1 "PESD12VS2UT" H 4700 4575 50  0000 C CNN
 F 2 "Package_TO_SOT_SMD:SOT-23" H 4700 4475 50  0001 C CNN
@@
 	4350 4150 5225 4150
 $Comp
-L power:GND #PWR?
+L power:GND #PWR080
 U 1 1 5F79653C
 P 4700 4675
-F 0 "#PWR?" H 4700 4425 50  0001 C CNN
+F 0 "#PWR080" H 4700 4425 50  0001 C CNN
 F 1 "GND" H 4705 4502 50  0000 C CNN
 F 2 "" H 4700 4675 50  0001 C CNN
@@
 $EndComp
 $Comp
-L Connector_Generic:Conn_01x04 J?
+L Connector_Generic:Conn_01x04 J21
 U 1 1 5F7AC162
 P 5250 5600
-F 0 "J?" H 5225 5275 50  0000 C CNN
+F 0 "J21" H 5225 5275 50  0000 C CNN
 F 1 "DATA_UART" H 5325 5825 50  0000 C CNN
 F 2 "Connector_PinHeader_2.54mm:PinHeader_1x04_P2.54mm_Horizontal" H 5250 5600 50  0001 C CNN
@@
 	5475 5825 5475 5800
 $Comp
-L power:GND #PWR?
+L power:GND #PWR082
 U 1 1 5F7AC5CD
 P 5475 5825
-F 0 "#PWR?" H 5475 5575 50  0001 C CNN
+F 0 "#PWR082" H 5475 5575 50  0001 C CNN
 F 1 "GND" H 5480 5652 50  0000 C CNN
 F 2 "" H 5475 5825 50  0001 C CNN
@@
 P 6025 5900
 AR Path="/5F51A37F/5F7AEF18" Ref="D?"  Part="1"
-AR Path="/5F709561/5F7AEF18" Ref="D?"  Part="1"
-F 0 "D?" H 5925 5800 50  0000 C CNN
+AR Path="/5F709561/5F7AEF18" Ref="D12"  Part="1"
+F 0 "D12" H 5925 5800 50  0000 C CNN
 F 1 "PESD3V3S2UT" H 6025 6000 50  0000 C CNN
 F 2 "Package_TO_SOT_SMD:SOT-23" H 6025 5900 50  0001 C CNN
@@
 $EndComp
 $Comp
-L power:GND #PWR?
+L power:GND #PWR085
 U 1 1 5F7AEF22
 P 6025 6100
-F 0 "#PWR?" H 6025 5850 50  0001 C CNN
+F 0 "#PWR085" H 6025 5850 50  0001 C CNN
 F 1 "GND" H 6030 5927 50  0000 C CNN
 F 2 "" H 6025 6100 50  0001 C CNN
@@
 P 6650 4500
 AR Path="/5F51A37F/5F818BA4" Ref="D?"  Part="1"
-AR Path="/5F709561/5F818BA4" Ref="D?"  Part="1"
-F 0 "D?" H 6550 4400 50  0000 C CNN
+AR Path="/5F709561/5F818BA4" Ref="D13"  Part="1"
+F 0 "D13" H 6550 4400 50  0000 C CNN
 F 1 "PESD3V3S2UT" H 6650 4600 50  0000 C CNN
 F 2 "Package_TO_SOT_SMD:SOT-23" H 6650 4500 50  0001 C CNN
@@
 $EndComp
 $Comp
-L power:GND #PWR?
+L power:GND #PWR087
 U 1 1 5F818BAE
 P 6650 4700
-F 0 "#PWR?" H 6650 4450 50  0001 C CNN
+F 0 "#PWR087" H 6650 4450 50  0001 C CNN
 F 1 "GND" H 6655 4527 50  0000 C CNN
 F 2 "" H 6650 4700 50  0001 C CNN
