File: Main_Board/kicad_project/stepper_driver.sch (KiCad schematic (older format))
At the start: 14 parts

Commit message: schematic rev1 finished
Parts:
- gave numbers to parts that had none: 14

Commit message: main board: layout start, steppers done
Parts:
- J1: footprint Connector_PinHeader_2.54mm:PinHeader_1x04_P2.54mm_Horizontal -> LoaDy:Molex_70543-0003
Changed lines of the file:
@@
 $Descr A4 11693 8268
 encoding utf-8
-Sheet 4 10
+Sheet 2 10
 Title "Cube Main Board - Stepper driver"
 Date "2020-09-02"
@@
 AR Path="/5F4A9E34/5F47373A" Ref="U4"  Part="1"
 AR Path="/5F4AD05F/5F47373A" Ref="U?"  Part="1"
-F 0 "U3" H 5625 5364 50  0000 C CNN
+F 0 "U1" H 5625 5364 50  0000 C CNN
 F 1 "TMC2209" H 5625 5235 100 0000 C CNN
 F 2 "LoaDy:TMC2209-LA" H 5875 2775 50  0001 C CNN
@@
 AR Path="/5F4A9E34/5F474870" Ref="C28"  Part="1"
 AR Path="/5F4AD05F/5F474870" Ref="C?"  Part="1"
-F 0 "C19" H 4683 4854 50  0000 R CNN
+F 0 "C1" H 4683 4854 50  0000 R CNN
 F 1 "100n" H 4683 4945 50  0000 R CNN
 F 2 "Capacitor_SMD:C_0603_1608Metric" H 4775 4900 50  0001 C CNN
@@
 AR Path="/5F4A9E34/5F4767FD" Ref="#PWR031"  Part="1"
 AR Path="/5F4AD05F/5F4767FD" Ref="#PWR?"  Part="1"
-F 0 "#PWR028" H 4775 4750 50  0001 C CNN
+F 0 "#PWR022" H 4775 4750 50  0001 C CNN
 F 1 "GND" H 4780 4827 50  0000 C CNN
 F 2 "" H 4775 5000 50  0001 C CNN
@@
 AR Path="/5F4A9E34/5F47FEA7" Ref="J4"  Part="1"
 AR Path="/5F4AD05F/5F47FEA7" Ref="J?"  Part="1"
-F 0 "J3" H 6980 2917 50  0000 L CNN
+F 0 "J1" H 6980 2917 50  0000 L CNN
 F 1 "MOTOR" H 6980 2826 50  0000 L CNN
-F 2 "Connector_PinHeader_2.54mm:PinHeader_1x04_P2.54mm_Horizontal" H 6900 2925 50  0001 C CNN
+F 2 "LoaDy:Molex_70543-0003" H 6900 2925 50  0001 C CNN
 F 3 "~" H 6900 2925 50  0001 C CNN
 	1    6900 2925
@@
 AR Path="/5F4A9E34/5F4817C7" Ref="C29"  Part="1"
 AR Path="/5F4AD05F/5F4817C7" Ref="C?"  Part="1"
-F 0 "C20" H 6517 3521 50  0000 L CNN
+F 0 "C2" H 6517 3521 50  0000 L CNN
 F 1 "100n" H 6517 3430 50  0000 L CNN
 F 2 "Capacitor_SMD:C_0603_1608Metric" H 6425 3475 50  0001 C CNN
@@
 AR Path="/5F4A9E34/5F482BEA" Ref="R7"  Part="1"
 AR Path="/5F4AD05F/5F482BEA" Ref="R?"  Part="1"
-F 0 "R5" V 6425 4350 50  0000 C CNN
+F 0 "R1" V 6425 4350 50  0000 C CNN
 F 1 "150m" V 6425 4575 50  0000 C CNN
 F 2 "Resistor_SMD:R_1206_3216Metric" H 6500 4425 50  0001 C CNN
@@
 AR Path="/5F4A9E34/5F484BD0" Ref="R8"  Part="1"
 AR Path="/5F4AD05F/5F484BD0" Ref="R?"  Part="1"
-F 0 "R6" V 6425 4425 50  0000 C CNN
+F 0 "R2" V 6425 4425 50  0000 C CNN
 F 1 "150m" V 6425 4675 50  0000 C CNN
 F 2 "Resistor_SMD:R_1206_3216Metric" H 6500 4525 50  0001 C CNN
@@
 AR Path="/5F4A9E34/5F485D07" Ref="#PWR032"  Part="1"
 AR Path="/5F4AD05F/5F485D07" Ref="#PWR?"  Part="1"
-F 0 "#PWR029" H 6850 4775 50  0001 C CNN
+F 0 "#PWR023" H 6850 4775 50  0001 C CNN
 F 1 "GND" H 6855 4852 50  0000 C CNN
 F 2 "" H 6850 5025 50  0001 C CNN
@@
 AR Path="/5F4A9E34/5F486EBD" Ref="C31"  Part="1"
 AR Path="/5F4AD05F/5F486EBD" Ref="C?"  Part="1"
-F 0 "C22" H 6942 4446 50  0000 L CNN
+F 0 "C4" H 6942 4446 50  0000 L CNN
 F 1 "2u2" H 6942 4355 50  0000 L CNN
 F 2 "Capacitor_SMD:C_0603_1608Metric" H 6850 4400 50  0001 C CNN
@@
 AR Path="/5F4A9E34/5F48B86C" Ref="C30"  Part="1"
 AR Path="/5F4AD05F/5F48B86C" Ref="C?"  Part="1"
-F 0 "C21" H 6592 4021 50  0000 L CNN
+F 0 "C3" H 6592 4021 50  0000 L CNN
 F 1 "22n" H 6592 3930 50  0000 L CNN
 F 2 "Capacitor_SMD:C_0603_1608Metric" H 6500 3975 50  0001 C CNN
@@
 AR Path="/5F4A9E34/5F48E2EC" Ref="C32"  Part="1"
 AR Path="/5F4AD05F/5F48E2EC" Ref="C?"  Part="1"
-F 0 "C23" H 7075 3875 50  0000 L CNN
+F 0 "C5" H 7075 3875 50  0000 L CNN
 F 1 "100n" H 7075 3725 50  0000 L CNN
 F 2 "Capacitor_SMD:C_0603_1608Metric" H 7025 3800 50  0001 C CNN
@@
 AR Path="/5F4A9E34/5F48E6B0" Ref="C33"  Part="1"
 AR Path="/5F4AD05F/5F48E6B0" Ref="C?"  Part="1"
-F 0 "C24" H 7350 3875 50  0000 L CNN
+F 0 "C6" H 7350 3875 50  0000 L CNN
 F 1 "100n" H 7350 3725 50  0000 L CNN
 F 2 "Capacitor_SMD:C_0603_1608Metric" H 7300 3800 50  0001 C CNN
@@
 AR Path="/5F4A9E34/5F48FB21" Ref="C36"  Part="1"
 AR Path="/5F4AD05F/5F48FB21" Ref="C?"  Part="1"
-F 0 "C27" H 8175 3875 50  0000 L CNN
+F 0 "C9" H 8175 3875 50  0000 L CNN
 F 1 "100u" H 8175 3725 50  0000 L CNN
 F 2 "Capacitor_SMD:CP_Elec_8x10" H 8125 3800 50  0001 C CNN
@@
 AR Path="/5F4A9E34/5F49697D" Ref="#PWR033"  Part="1"
 AR Path="/5F4AD05F/5F49697D" Ref="#PWR?"  Part="1"
-F 0 "#PWR030" H 8125 3750 50  0001 C CNN
+F 0 "#PWR024" H 8125 3750 50  0001 C CNN
 F 1 "GND" H 8130 3827 50  0000 C CNN
 F 2 "" H 8125 4000 50  0001 C CNN
@@
 AR Path="/5F4A9E34/5F49B00A" Ref="C34"  Part="1"
 AR Path="/5F4AD05F/5F49B00A" Ref="C?"  Part="1"
-F 0 "C25" H 7625 3875 50  0000 L CNN
+F 0 "C7" H 7625 3875 50  0000 L CNN
 F 1 "10u" H 7600 3725 50  0000 L CNN
 F 2 "Capacitor_SMD:C_1210_3225Metric" H 7575 3800 50  0001 C CNN
@@
 AR Path="/5F4A9E34/5F49B360" Ref="C35"  Part="1"
 AR Path="/5F4AD05F/5F49B360" Ref="C?"  Part="1"
-F 0 "C26" H 7900 3875 50  0000 L CNN
+F 0 "C8" H 7900 3875 50  0000 L CNN
 F 1 "10u" H 7875 3725 50  0000 L CNN
 F 2 "Capacitor_SMD:C_1210_3225Metric" H 7850 3800 50  0001 C CNN
@@
 AR Path="/5F4A9CF3/5F51F4C4" Ref="TP3"  Part="1"
 AR Path="/5F4A9E34/5F51F4C4" Ref="TP4"  Part="1"
-F 0 "TP3" V 4350 2225 50  0000 R CNN
+F 0 "TP1" V 4350 2225 50  0000 R CNN
 F 1 "DRIVER_TP" V 4250 2225 50  0000 R CNN
 F 2 "Connector_PinHeader_2.54mm:PinHeader_1x05_P2.54mm_Vertical" H 4300 2525 50  0001 C CNN

Commit message: Main board sch: add backup battery, update license
Changed lines of the file:
@@
 Rev "1"
 Comp "Oldřich Pecák (LoaDy)"
-Comment1 "Licensed under CERN-OHL-P v2"
+Comment1 "Licensed under CERN-OHL-W v2"
 Comment2 ""
 Comment3 ""
@@
 AR Path="/5F4A9E34/5F47373A" Ref="U4"  Part="1"
 AR Path="/5F4AD05F/5F47373A" Ref="U?"  Part="1"
-F 0 "U1" H 5625 5364 50  0000 C CNN
+F 0 "U4" H 5625 5364 50  0000 C CNN
 F 1 "TMC2209" H 5625 5235 100 0000 C CNN
 F 2 "LoaDy:TMC2209-LA" H 5875 2775 50  0001 C CNN
@@
 AR Path="/5F4A9E34/5F474870" Ref="C28"  Part="1"
 AR Path="/5F4AD05F/5F474870" Ref="C?"  Part="1"
-F 0 "C1" H 4683 4854 50  0000 R CNN
+F 0 "C28" H 4683 4854 50  0000 R CNN
 F 1 "100n" H 4683 4945 50  0000 R CNN
 F 2 "Capacitor_SMD:C_0603_1608Metric" H 4775 4900 50  0001 C CNN
@@
 AR Path="/5F4A9E34/5F47FEA7" Ref="J4"  Part="1"
 AR Path="/5F4AD05F/5F47FEA7" Ref="J?"  Part="1"
-F 0 "J1" H 6980 2917 50  0000 L CNN
+F 0 "J4" H 6980 2917 50  0000 L CNN
 F 1 "MOTOR" H 6980 2826 50  0000 L CNN
 F 2 "LoaDy:Molex_70543-0003" H 6900 2925 50  0001 C CNN
@@
 AR Path="/5F4A9E34/5F4817C7" Ref="C29"  Part="1"
 AR Path="/5F4AD05F/5F4817C7" Ref="C?"  Part="1"
-F 0 "C2" H 6517 3521 50  0000 L CNN
+F 0 "C29" H 6517 3521 50  0000 L CNN
 F 1 "100n" H 6517 3430 50  0000 L CNN
 F 2 "Capacitor_SMD:C_0603_1608Metric" H 6425 3475 50  0001 C CNN
@@
 AR Path="/5F4A9E34/5F482BEA" Ref="R7"  Part="1"
 AR Path="/5F4AD05F/5F482BEA" Ref="R?"  Part="1"
-F 0 "R1" V 6425 4350 50  0000 C CNN
+F 0 "R7" V 6425 4350 50  0000 C CNN
 F 1 "150m" V 6425 4575 50  0000 C CNN
 F 2 "Resistor_SMD:R_1206_3216Metric" H 6500 4425 50  0001 C CNN
@@
 AR Path="/5F4A9E34/5F484BD0" Ref="R8"  Part="1"
 AR Path="/5F4AD05F/5F484BD0" Ref="R?"  Part="1"
-F 0 "R2" V 6425 4425 50  0000 C CNN
+F 0 "R8" V 6425 4425 50  0000 C CNN
 F 1 "150m" V 6425 4675 50  0000 C CNN
 F 2 "Resistor_SMD:R_1206_3216Metric" H 6500 4525 50  0001 C CNN
@@
 AR Path="/5F4A9E34/5F486EBD" Ref="C31"  Part="1"
 AR Path="/5F4AD05F/5F486EBD" Ref="C?"  Part="1"
-F 0 "C4" H 6942 4446 50  0000 L CNN
+F 0 "C31" H 6942 4446 50  0000 L CNN
 F 1 "2u2" H 6942 4355 50  0000 L CNN
 F 2 "Capacitor_SMD:C_0603_1608Metric" H 6850 4400 50  0001 C CNN
@@
 AR Path="/5F4A9E34/5F48B86C" Ref="C30"  Part="1"
 AR Path="/5F4AD05F/5F48B86C" Ref="C?"  Part="1"
-F 0 "C3" H 6592 4021 50  0000 L CNN
+F 0 "C30" H 6592 4021 50  0000 L CNN
 F 1 "22n" H 6592 3930 50  0000 L CNN
 F 2 "Capacitor_SMD:C_0603_1608Metric" H 6500 3975 50  0001 C CNN
@@
 AR Path="/5F4A9E34/5F48E2EC" Ref="C32"  Part="1"
 AR Path="/5F4AD05F/5F48E2EC" Ref="C?"  Part="1"
-F 0 "C5" H 7075 3875 50  0000 L CNN
+F 0 "C32" H 7075 3875 50  0000 L CNN
 F 1 "100n" H 7075 3725 50  0000 L CNN
 F 2 "Capacitor_SMD:C_0603_1608Metric" H 7025 3800 50  0001 C CNN
@@
 AR Path="/5F4A9E34/5F48E6B0" Ref="C33"  Part="1"
 AR Path="/5F4AD05F/5F48E6B0" Ref="C?"  Part="1"
-F 0 "C6" H 7350 3875 50  0000 L CNN
+F 0 "C33" H 7350 3875 50  0000 L CNN
 F 1 "100n" H 7350 3725 50  0000 L CNN
 F 2 "Capacitor_SMD:C_0603_1608Metric" H 7300 3800 50  0001 C CNN
@@
 AR Path="/5F4A9E34/5F48FB21" Ref="C36"  Part="1"
 AR Path="/5F4AD05F/5F48FB21" Ref="C?"  Part="1"
-F 0 "C9" H 8175 3875 50  0000 L CNN
+F 0 "C36" H 8175 3875 50  0000 L CNN
 F 1 "100u" H 8175 3725 50  0000 L CNN
 F 2 "Capacitor_SMD:CP_Elec_8x10" H 8125 3800 50  0001 C CNN
@@
 AR Path="/5F4A9E34/5F49B00A" Ref="C34"  Part="1"
 AR Path="/5F4AD05F/5F49B00A" Ref="C?"  Part="1"
-F 0 "C7" H 7625 3875 50  0000 L CNN
+F 0 "C34" H 7625 3875 50  0000 L CNN
 F 1 "10u" H 7600 3725 50  0000 L CNN
 F 2 "Capacitor_SMD:C_1210_3225Metric" H 7575 3800 50  0001 C CNN
@@
 AR Path="/5F4A9E34/5F49B360" Ref="C35"  Part="1"
 AR Path="/5F4AD05F/5F49B360" Ref="C?"  Part="1"
-F 0 "C8" H 7900 3875 50  0000 L CNN
+F 0 "C35" H 7900 3875 50  0000 L CNN
 F 1 "10u" H 7875 3725 50  0000 L CNN
 F 2 "Capacitor_SMD:C_1210_3225Metric" H 7850 3800 50  0001 C CNN
@@
 AR Path="/5F4A9CF3/5F51F4C4" Ref="TP3"  Part="1"
 AR Path="/5F4A9E34/5F51F4C4" Ref="TP4"  Part="1"
-F 0 "TP1" V 4350 2225 50  0000 R CNN
+F 0 "TP4" V 4350 2225 50  0000 R CNN
 F 1 "DRIVER_TP" V 4250 2225 50  0000 R CNN
 F 2 "Connector_PinHeader_2.54mm:PinHeader_1x05_P2.54mm_Vertical" H 4300 2525 50  0001 C CNN
