File: main_board/kicad_project/expansion.sch (KiCad schematic (older format))
At the start: 24 parts, among them J24 EXPANSION_HEADER

Commit message: change resistor network package
Parts:
- RN1, RN2, RN3, RN4, RN5, RN6, RN7, RN8: footprint Resistor_SMD:R_Array_Convex_4x1206 -> Resistor_SMD:R_Array_Convex_4x0603
Changed lines of the file:
@@
 Sheet 10 10
 Title "Cube Main Board - Expansion Header"
-Date "2020-09-26"
-Rev "1.1"
+Date "2021-03-13"
+Rev "1.2"
 Comp "Oldřich Pecák (LoaDy)"
 Comment1 "Licensed under CERN-OHL-W v2"
@@
 F 0 "RN1" V 5150 4100 50  0000 C CNN
 F 1 "150R" V 5150 4325 50  0000 C CNN
-F 2 "Resistor_SMD:R_Array_Convex_4x1206" V 5725 4225 50  0001 C CNN
+F 2 "Resistor_SMD:R_Array_Convex_4x0603" V 5725 4225 50  0001 C CNN
 F 3 "~" H 5450 4225 50  0001 C CNN
 	1    5450 4225
@@
 F 0 "RN2" V 5150 4600 50  0000 C CNN
 F 1 "150R" V 5150 4825 50  0000 C CNN
-F 2 "Resistor_SMD:R_Array_Convex_4x1206" V 5725 4725 50  0001 C CNN
+F 2 "Resistor_SMD:R_Array_Convex_4x0603" V 5725 4725 50  0001 C CNN
 F 3 "~" H 5450 4725 50  0001 C CNN
 	1    5450 4725
@@
 F 0 "RN3" V 5150 5100 50  0000 C CNN
 F 1 "150R" V 5150 5325 50  0000 C CNN
-F 2 "Resistor_SMD:R_Array_Convex_4x1206" V 5725 5225 50  0001 C CNN
+F 2 "Resistor_SMD:R_Array_Convex_4x0603" V 5725 5225 50  0001 C CNN
 F 3 "~" H 5450 5225 50  0001 C CNN
 	1    5450 5225
@@
 F 0 "RN4" V 5150 5600 50  0000 C CNN
 F 1 "150R" V 5150 5825 50  0000 C CNN
-F 2 "Resistor_SMD:R_Array_Convex_4x1206" V 5725 5725 50  0001 C CNN
+F 2 "Resistor_SMD:R_Array_Convex_4x0603" V 5725 5725 50  0001 C CNN
 F 3 "~" H 5450 5725 50  0001 C CNN
 	1    5450 5725
@@
 F 0 "RN8" V 7025 5225 50  0000 C CNN
 F 1 "150R" V 7025 5425 50  0000 C CNN
-F 2 "Resistor_SMD:R_Array_Convex_4x1206" V 7600 5325 50  0001 C CNN
+F 2 "Resistor_SMD:R_Array_Convex_4x0603" V 7600 5325 50  0001 C CNN
 F 3 "~" H 7325 5325 50  0001 C CNN
 	1    7325 5325
@@
 F 0 "RN7" V 7025 4725 50  0000 C CNN
 F 1 "150R" V 7025 4925 50  0000 C CNN
-F 2 "Resistor_SMD:R_Array_Convex_4x1206" V 7600 4825 50  0001 C CNN
+F 2 "Resistor_SMD:R_Array_Convex_4x0603" V 7600 4825 50  0001 C CNN
 F 3 "~" H 7325 4825 50  0001 C CNN
 	1    7325 4825
@@
 F 0 "RN6" V 7025 4225 50  0000 C CNN
 F 1 "150R" V 7025 4425 50  0000 C CNN
-F 2 "Resistor_SMD:R_Array_Convex_4x1206" V 7600 4325 50  0001 C CNN
+F 2 "Resistor_SMD:R_Array_Convex_4x0603" V 7600 4325 50  0001 C CNN
 F 3 "~" H 7325 4325 50  0001 C CNN
 	1    7325 4325
@@
 F 0 "RN5" V 7025 3725 50  0000 C CNN
 F 1 "150R" V 7025 3925 50  0000 C CNN
-F 2 "Resistor_SMD:R_Array_Convex_4x1206" V 7600 3825 50  0001 C CNN
+F 2 "Resistor_SMD:R_Array_Convex_4x0603" V 7600 3825 50  0001 C CNN
 F 3 "~" H 7325 3825 50  0001 C CNN
 	1    7325 3825
